Commit message: Updated actual robot start position

File: urdf/kuka_iiwa_1.urdf (robot description, URDF)
Before this commit: robot lbr_iiwa, 11 links, 10 joints
Joints:
- joint base_link_to_chassis: origin xyz=0.8839 -0.3889 -0.42 rpy=0 0 3.9270 -> xyz=-0.8839 -0.3889 -0.42 rpy=0 0 1.57

File: urdf/kuka_iiwa_2.urdf (robot description, URDF)
Before this commit: robot lbr_iiwa, 11 links, 10 joints
Joints:
- joint base_link_to_chassis: origin xyz=-0.8839 0.3889 -0.42 rpy=0 0 0.7854 -> xyz=0.9 0.23984 -0.42 rpy=0 0 -1.57
